File: hardware/gdt/gdt.sch (KiCad schematic (older format))
At the start: 28 parts, among them J1 USB_OTG, J2 USB_A, Q1 Q_NPN_BEC, Q2 Q_NPN_BEC, Q3 Q_NMOS_GDS, U1 CH340G, U2 AP1117-33, U3 ESP-12E, Y1 12M

Commit message: Whoops; this put it into boot mode 5 during reset rather than 1 -- forgot a pulldown resistor.
Parts:
- added R13: 10k, coddingtonbear/coddingtonbear.pretty:0805_Milling, symbol R
Connections:
- net GND: now also R13.1
- net at Q3.1 (G), U3.16 (GPIO15): now also R13.2
Changed lines of the file:
@@
 Text GLabel 5100 4550 1    60   BiDi ~ 0
 REST
+$Comp
+L R R13
+U 1 1 59E9A93D
+P 8050 5550
+F 0 "R13" V 7843 5550 50  0000 C CNN
+F 1 "10k" V 7934 5550 50  0000 C CNN
+F 2 "coddingtonbear/coddingtonbear.pretty:0805_Milling" V 7980 5550 50  0001 C CNN
+F 3 "" H 8050 5550 50  0001 C CNN
+	1    8050 5550
+	-1   0    0    1
+$EndComp
+$Comp
+L GND #PWR022
+U 1 1 59E9A9C5
+P 8050 5700
+F 0 "#PWR022" H 8050 5450 50  0001 C CNN
+F 1 "GND" H 8055 5527 50  0000 C CNN
+F 2 "" H 8050 5700 50  0001 C CNN
+F 3 "" H 8050 5700 50  0001 C CNN
+	1    8050 5700
+	1    0    0    -1
+$EndComp
 $EndSCHEMATC

Commit message: Uploading final version of hardware/software.
Parts:
- removed Q3: Q_NMOS_GDS, cpavlina/kicad-pcblib/pth-semi.pretty:TO-220, symbol Q_NMOS_GDS
Connections:
- net +5V: now also J2.1 (VBUS)
Changed lines of the file:
@@
 L +5V #PWR04
 U 1 1 59E588B7
-P 9600 5700
-F 0 "#PWR04" H 9600 5550 50  0001 C CNN
-F 1 "+5V" H 9615 5873 50  0000 C CNN
-F 2 "" H 9600 5700 50  0001 C CNN
-F 3 "" H 9600 5700 50  0001 C CNN
-	1    9600 5700
+P 10050 4700
+F 0 "#PWR04" H 10050 4550 50  0001 C CNN
+F 1 "+5V" H 10065 4873 50  0000 C CNN
+F 2 "" H 10050 4700 50  0001 C CNN
+F 3 "" H 10050 4700 50  0001 C CNN
+	1    10050 4700
 	-1   0    0    1
 $EndComp
@@
 Wire Wire Line
 	900  2500 1050 2500
-$Comp
-L R R6
-U 1 1 59E5DACD
-P 7050 4100
-F 0 "R6" V 6843 4100 50  0000 C CNN
-F 1 "JMP_D-" V 6934 4100 50  0000 C CNN
-F 2 "coddingtonbear/coddingtonbear.pretty:0805_Milling" V 6980 4100 50  0001 C CNN
-F 3 "" H 7050 4100 50  0001 C CNN
-	1    7050 4100
-	0    1    1    0
-$EndComp
-$Comp
-L R R7
-U 1 1 59E5DBD0
-P 7050 4300
-F 0 "R7" V 6843 4300 50  0000 C CNN
-F 1 "JMP_D+" V 6934 4300 50  0000 C CNN
-F 2 "coddingtonbear/coddingtonbear.pretty:0805_Milling" V 6980 4300 50  0001 C CNN
-F 3 "" H 7050 4300 50  0001 C CNN
-	1    7050 4300
-	0    1    1    0
-$EndComp
-Wire Wire Line
-	5300 4650 5450 4650
-Wire Wire Line
-	5300 4100 5300 4650
-Wire Wire Line
-	5300 4300 6900 4300
-Wire Wire Line
-	6900 4100 5300 4100
-Connection ~ 5300 4300
-Wire Wire Line
-	7200 4300 8200 4300
-Wire Wire Line
-	8200 4300 8200 4500
 Connection ~ 8200 4500
-Wire Wire Line
-	7200 4100 8300 4100
-Wire Wire Line
-	8300 4100 8300 4400
 Connection ~ 8300 4400
 $Comp
@@
 Wire Wire Line
 	7950 4750 7350 4750
-$Comp
-L Q_NMOS_GDS Q3
-U 1 1 59E6248B
-P 9500 5400
-F 0 "Q3" H 9705 5354 50  0000 L CNN
-F 1 "Q_NMOS_GDS" H 9705 5445 50  0000 L CNN
-F 2 "cpavlina/kicad-pcblib/pth-semi.pretty:TO-220" H 9700 5500 50  0001 C CNN
-F 3 "" H 9500 5400 50  0001 C CNN
-	1    9500 5400
-	1    0    0    1
-$EndComp
-Wire Wire Line
-	9600 5700 9600 5600
-Wire Wire Line
-	9600 5200 9600 4950
-Wire Wire Line
-	9600 4950 10050 4950
-Wire Wire Line
-	10050 4950 10050 4700
-Wire Wire Line
-	9300 5400 8050 5400
 Wire Wire Line
 	8050 5400 8050 5150
@@
 	1    0    0    -1
 $EndComp
+Wire Wire Line
+	8300 4100 8300 4400
+Wire Wire Line
+	8200 4300 8200 4500
+Wire Wire Line
+	7200 4300 8200 4300
+Wire Wire Line
+	7200 4100 8300 4100
+Wire Wire Line
+	5300 4650 5450 4650
+Wire Wire Line
+	6900 4100 5300 4100
+Connection ~ 5300 4300
+Wire Wire Line
+	5300 4100 5300 4650
+Wire Wire Line
+	5300 4300 6900 4300
+$Comp
+L R R7
+U 1 1 59E5DBD0
+P 7050 4300
+F 0 "R7" V 6843 4300 50  0000 C CNN
+F 1 "JMP_D+" V 6934 4300 50  0000 C CNN
+F 2 "coddingtonbear/coddingtonbear.pretty:0805_Milling" V 6980 4300 50  0001 C CNN
+F 3 "" H 7050 4300 50  0001 C CNN
+	1    7050 4300
+	0    1    1    0
+$EndComp
+$Comp
+L R R6
+U 1 1 59E5DACD
+P 7050 4100
+F 0 "R6" V 6843 4100 50  0000 C CNN
+F 1 "JMP_D-" V 6934 4100 50  0000 C CNN
+F 2 "coddingtonbear/coddingtonbear.pretty:0805_Milling" V 6980 4100 50  0001 C CNN
+F 3 "" H 7050 4100 50  0001 C CNN
+	1    7050 4100
+	0    1    1    0
+$EndComp
 $EndSCHEMATC
